File: Arduino/PCB/Ext_Arduino01/ADC_MCPV01.kicad_pcb (KiCad board)
At the start: 2 copper layers, 78.7 x 65.5 mm, 57 parts, among them J1 Conn_01x04, J10 Ard23_32, J11 Skt01_08, J12 Skt15_22, J13 Skt09_14, J14 Skt23_32, J15 P01, J16 P02, J17 P03, J18 P04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

Commit message: actualizando kicad
Parts:
- moved J5 5.08 mm to (108.2, 48.3), turned to -90 degrees
- moved D8 3.05 mm to (103.1, 60.6)
- moved R11 2.03 mm to (104.1, 65.5)
Connections:
- J5 pad 1: Net-(J5-Pin_1) -> Net-(D6-K)
- J5 pad 2: Net-(D6-K) -> Net-(J5-Pin_2)
- JP_VDC1 pad 1: Net-(J5-Pin_1) -> Net-(J5-Pin_2)
- R10 pad 2: Net-(J5-Pin_1) -> Net-(J5-Pin_2)
Routing:
- net Net-(J5-Pin_2): track 0.00 -> 36.7 mm
- net Net-(J5-Pin_1): track 36.7 -> 0.00 mm
- net INO06: track 300.7 -> 307.0 mm
- net INO15: track 19.1 -> 19.9 mm
- added copper zone on B.Cu, net INO06
- added copper zone on F.Cu, net INO06
Other:
- board text added: "- +"
- board text added: "12V - + Ext"
- board text added: "Reg 6V"
- board text added: "https://github.com/faiverht/Proyecto-HFH"
- board text removed: "+ -"
- board text removed: "12V + - Ext"
- board text removed: "6V"
