File: Arduino/PCB/Ext_Arduino01/ADC_MCPV01.kicad_sch (KiCad schematic)
At the start: 54 parts, among them J1 Conn_01x04, J10 Ard23_32, J11 Skt01_08, J12 Skt15_22, J13 Skt09_14, J14 Skt23_32, J15 P01, J16 P02, J17 P03, J18 P04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

Commit message: actualizando kicad
Connections:
- net at JP_VDC1.1 (A), R10.2: now also J5.2 (Pin_2); no longer J5.1 (Pin_1)
- net at D6.1 (K), J6.3: now also J5.1 (Pin_1); no longer J5.2 (Pin_2)
Other:
- moved on the sheet: J5
Changed lines of the file:
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@@
   (junction (at 30.48 110.49) (diameter 0) (color 0 0 0 0)
   )
-  (junction (at 43.18 110.49) (diameter 0) (color 0 0 0 0)
-  )
   (junction (at 104.14 26.67) (diameter 0) (color 0 0 0 0)
   )
+  (junction (at 43.18 110.49) (diameter 0) (color 0 0 0 0)
+  )
   (junction (at 48.26 88.9) (diameter 0) (color 0 0 0 0)
   )
@@
     (stroke (width 0) (type default))
   )
+  (wire (pts (xy 111.76 29.21) (xy 111.76 44.45))
+    (stroke (width 0) (type default))
+  )
   (wire (pts (xy 20.32 48.26) (xy 20.32 52.07))
     (stroke (width 0) (type default))
@@
     (stroke (width 0) (type default))
   )
-  (wire (pts (xy 100.33 29.21) (xy 111.76 29.21))
-    (stroke (width 0) (type default))
-  )
   (wire (pts (xy 59.69 96.52) (xy 71.12 96.52))
     (stroke (width 0) (type default))
@@
     (stroke (width 0) (type default))
   )
+  (wire (pts (xy 100.33 29.21) (xy 111.76 29.21))
+    (stroke (width 0) (type default))
+  )
   (wire (pts (xy 175.26 40.64) (xy 176.53 40.64))
     (stroke (width 0) (type default))
@@
     (stroke (width 0) (type default))
   )
-  (wire (pts (xy 111.76 29.21) (xy 111.76 44.45))
-    (stroke (width 0) (type default))
-  )
   (wire (pts (xy 111.76 44.45) (xy 128.27 44.45))
     (stroke (width 0) (type default))
@@
     (stroke (width 0) (type default))
   )
+  (wire (pts (xy 100.33 26.67) (xy 104.14 26.67))
+    (stroke (width 0) (type default))
+  )
   (wire (pts (xy 34.29 165.1) (xy 35.56 165.1))
     (stroke (width 0) (type default))
@@
     (stroke (width 0) (type default))
   )
-  (wire (pts (xy 100.33 26.67) (xy 104.14 26.67))
-    (stroke (width 0) (type default))
-  )
   (wire (pts (xy 208.28 30.48) (xy 209.55 30.48))
     (stroke (width 0) (type default))
@@
     )
   )
-  (symbol (lib_id "Connector_Generic:Conn_01x02") (at 95.25 26.67 0) (mirror y) (unit 1)
+  (symbol (lib_id "Connector_Generic:Conn_01x02") (at 95.25 29.21 180) (unit 1)
     (exclude_from_sim no) (in_bom yes) (on_board yes) (dnp no)
-    (property "Reference" "J5" (at 96.52 23.622 0)
+    (property "Reference" "J5" (at 96.52 32.258 0)
       (effects (font (size 1.27 1.27)) (justify left))
     )
@@
       (effects (font (size 1.27 1.27)) (justify left))
     )
-    (property "Footprint" "TerminalBlock_Phoenix:TerminalBlock_Phoenix_MKDS-1,5-2-5.08_1x02_P5.08mm_Horizontal" (at 95.25 26.67 0)
+    (property "Footprint" "TerminalBlock_Phoenix:TerminalBlock_Phoenix_MKDS-1,5-2-5.08_1x02_P5.08mm_Horizontal" (at 95.25 29.21 0)
       (effects (font (size 1.27 1.27)) hide)
     )
-    (property "Datasheet" "~" (at 95.25 26.67 0)
+    (property "Datasheet" "~" (at 95.25 29.21 0)
       (effects (font (size 1.27 1.27)) hide)
     )
-    (property "Description" "Generic connector, single row, 01x02, script generated (kicad-library-utils/schlib/autogen/connector/)" (at 95.25 26.67 0)
+    (property "Description" "Generic connector, single row, 01x02, script generated (kicad-library-utils/schlib/autogen/connector/)" (at 95.25 29.21 0)
       (effects (font (size 1.27 1.27)) hide)
     )
